File: camera_base/camera_base.kicad_pcb (KiCad board)
At the start: 2 copper layers, 100 x 80 mm, 19 parts, among them J1 Raspberry_Pi_4, J2 Conn_02x03_Odd_Even, SW1 SW_Push_Dual, SW2 SW_Push_Dual, SW3 SW_Push_Dual, SW5 SW_Push_Dual

Commit message: aesthetics
Parts:
- RV1: moved to B.Cu
- moved H2 1.25 mm to (157.0, 63.0)
- turned RV1 to 180 degrees
Other:
- board text added: "01"
- board text added: "18"
- board text added: "23"
- board text added: "24"
- board text added: "25"
- board text added: "BREAKOUTS"
- board text added: "CAPTURE"
- board text added: "GPIO"
- board text added: "GPIO_04"
- board text added: "GPIO_12"
- board text added: "GPIO_26"
- board text added: "MODEL / ID"
- board text added: "NON_OPTIMAL_CAMERA"
- board text added: "PLAYBACK"
- board text added: "V1"
- board text removed: "BREAKOUT"
- board text removed: "MODEL"
- board text removed: "NON_OPTIMAL CAMERA v1"
- board text removed: "SHOOT"
- board text removed: "VIEW"
