File: camera_base/camera_base.kicad_sch (KiCad schematic)
At the start: 15 parts, among them J1 Raspberry_Pi_4, J2 Conn_02x06_Odd_Even, SW1 SW_Push_Dual, SW2 SW_Push_Dual, SW3 SW_Push_Dual, SW4 SW_Push_Dual, SW5 SW_Push_Dual

Commit message: update
Parts:
- removed J2: Conn_02x06_Odd_Even, Connector_PinSocket_2.54mm:PinSocket_2x06_P2.54mm_Vertical, symbol Connector_Generic:Conn_02x06_Odd_Even
- removed SW4: SW_Push_Dual, camera_base:PUSH_BUTTON_12mm, symbol Switch:SW_Push_Dual
- added D1, D2: LED, LED_THT:LED_D3.0mm, symbol Device:LED
- added J2: Conn_02x03_Odd_Even, Connector_PinHeader_2.54mm:PinHeader_2x03_P2.54mm_Vertical, symbol Connector_Generic:Conn_02x03_Odd_Even
- added R1, R2: R, Resistor_THT:R_Axial_DIN0204_L3.6mm_D1.6mm_P5.08mm_Vertical, symbol Device:R
- added RV1: R_Potentiometer_US, Potentiometer_THT:Potentiometer_Alps_RK163_Single_Horizontal, symbol Device:R_Potentiometer_US
Connections:
- net 3v3: now also J1.17 (3V3), RV1.1
- net CE0: now also TFT1.7 (TFTCS); no longer TFT1.10 (SDCS)
- net CE1: now also TFT1.10 (SDCS); no longer TFT1.7 (TFTCS)
- net GND: now also J1.25 (GND), J1.9 (GND), D1.1 (K), D2.1 (K), J2.2 (Pin_2), J2.4 (Pin_4), J2.6 (Pin_6), RV1.3
- net GPIO_01: now also S4.1 (A); no longer S4.3 (C)
- net GPIO_13: now also R2.1; no longer SW3.1
- net GPIO_14: no longer J1.8 (GPIO14/UART_TXD), TFT1.8 (RST)
- net GPIO_15: no longer TFT1.9 (DC)
- net GPIO_16: now also TFT1.11 (LIT); no longer S4.6 (CENTER)
- net GPIO_18: now also S4.5 (D); no longer TFT1.11 (LIT)
- net GPIO_19: now also R1.1
- net GPIO_20: now also TFT1.9 (DC); no longer S4.5 (D)
- net GPIO_21: now also TFT1.8 (RST); no longer SW2.1
- net GPIO_23: now also S4.6 (CENTER); no longer SW1.1
- net GPIO_24: now also S4.3 (C); no longer S4.1 (A)
- net GPIO_02: now reaches J1.3 (SDA_I2C1/GPIO02)
- net GPIO_02: now also RV1.2
- net GPIO_22: now reaches J1.15 (GPIO22/SDIO_CLK)
- net GPIO_22: now also J2.1 (Pin_1)
- net GPIO_03: now reaches J1.5 (SCL_I2C1/GPIO03)
- net GPIO_03: now also SW3.1
- net GPIO_04: now reaches J1.7 (GPCLK0/GPIO04)
- net GPIO_04: now also SW2.1
- net GPIO_11: now reaches J1.11 (GPIO17/SPI1_~{CE1})
- net GPIO_11: now also J2.5 (Pin_5)
- net GPIO_27: now reaches J1.13 (GPIO27/SDIO_DAT3)
- net GPIO_27: now also J2.3 (Pin_3)
- net GPIO_12: now reaches J1.32 (GPIO12/PWM0)
- net GPIO_12: now also SW1.1
- new net: D1.2 (A), R1.2
- new net: D2.2 (A), R2.2
- no-connect marks 23 -> 19

Commit message: update
Other:
- moved on the sheet: D1, D2, H1, H2, H3, H4, J1, J2, POW1, R1, R2, RV1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
